Commit message: fixed urdf and added simulated short (robot without control and will collapse to the foor)

File: assets/mh5_revH.urdf (robot description, URDF)
Before this commit: robot mh5_robot, 28 links, 27 joints
Links:
- link chest: geometry collision mesh filename=package://mh5_description/meshes/chest_revH.stl; visual mesh filename=package://mh5_description/meshes/chest_revH.stl
- link head_frame: geometry collision mesh filename=package://mh5_description/meshes/head_revH.stl; visual mesh filename=package://mh5_description/meshes/head_revH.stl
- link head_servo: geometry collision mesh filename=package://mh5_description/meshes/2XL430_1_idle_revC.stl; visual mesh filename=package://mh5_description/meshes/2XL430_1_idle_revC.stl
- link left_ankle_servo: geometry collision mesh filename=package://mh5_description/meshes/2XL430_2_idles_revC.stl; visual mesh filename=package://mh5_description/meshes/2XL430_2_idles_revC.stl
- link left_elbow_frame: geometry collision mesh filename=package://mh5_description/meshes/frame02_revC.stl; visual mesh filename=package://mh5_description/meshes/frame02_revC.stl
- link left_foot: geometry collision mesh filename=package://mh5_description/meshes/foot_revH.stl; visual mesh filename=package://mh5_description/meshes/foot_revH.stl
- link left_gripper: geometry collision mesh filename=package://mh5_description/meshes/gripper.stl; visual mesh filename=package://mh5_description/meshes/gripper.stl
- link left_hip_servo: geometry collision mesh filename=package://mh5_description/meshes/2XL430_2_idles_revC.stl; visual mesh filename=package://mh5_description/meshes/2XL430_2_idles_revC.stl
- link left_knee_servo: geometry collision mesh filename=package://mh5_description/meshes/2XL430_1_idle_revC.stl; visual mesh filename=package://mh5_description/meshes/2XL430_1_idle_revC.stl
- link left_lower_arm: geometry collision mesh filename=package://mh5_description/meshes/left_lower_arm.stl; visual mesh filename=package://mh5_description/meshes/left_lower_arm.stl
- link left_shoulder_frame: geometry collision mesh filename=package://mh5_description/meshes/frame04_revE.stl; visual mesh filename=package://mh5_description/meshes/frame04_revE.stl
- link left_thigh: geometry collision mesh filename=package://mh5_description/meshes/thigh_revE.stl; visual mesh filename=package://mh5_description/meshes/thigh_revE.stl
- link left_tibia: geometry collision mesh filename=package://mh5_description/meshes/frame02_revC.stl; visual mesh filename=package://mh5_description/meshes/frame02_revC.stl
- link left_upper_arm: geometry collision mesh filename=package://mh5_description/meshes/upper_arm.stl; visual mesh filename=package://mh5_description/meshes/upper_arm.stl
- link right_elbow_frame: geometry collision mesh filename=package://mh5_description/meshes/frame02_revC.stl; visual mesh filename=package://mh5_description/meshes/frame02_revC.stl
- link right_foot: geometry collision mesh filename=package://mh5_description/meshes/foot_revH.stl; visual mesh filename=package://mh5_description/meshes/foot_revH.stl
- link right_gripper: geometry collision mesh filename=package://mh5_description/meshes/gripper.stl; visual mesh filename=package://mh5_description/meshes/gripper.stl
- link right_lower_arm: geometry collision mesh filename=package://mh5_description/meshes/right_lower_arm.stl; visual mesh filename=package://mh5_description/meshes/right_lower_arm.stl
- link right_shoulder_frame: geometry collision mesh filename=package://mh5_description/meshes/frame04_revE.stl; visual mesh filename=package://mh5_description/meshes/frame04_revE.stl
- link right_upper_arm: geometry collision mesh filename=package://mh5_description/meshes/upper_arm.stl; visual mesh filename=package://mh5_description/meshes/upper_arm.stl
Joints:
- joint chest_fixed: type fixed -> floating
