Commit message: reorg env defintion

File: envs/assets/mh5_revH.urdf (robot description, URDF)
Before this commit: robot mh5_robot, 28 links, 27 joints
Links:
- link chest: geometry collision mesh filename=package://mh5_description/meshes/chest_revH.dae; visual mesh filename=package://mh5_description/meshes/chest_revH.dae
- link head_frame: geometry collision mesh filename=package://mh5_description/meshes/head_revH.dae; visual mesh filename=package://mh5_description/meshes/head_revH.dae
- link left_foot: geometry collision mesh filename=package://mh5_description/meshes/foot_revH.dae; visual mesh filename=package://mh5_description/meshes/foot_revH.dae
- link left_gripper: geometry collision mesh filename=package://mh5_description/meshes/gripper.dae; visual mesh filename=package://mh5_description/meshes/gripper.dae
- link left_lower_arm: geometry collision mesh filename=package://mh5_description/meshes/left_lower_arm.dae; visual mesh filename=package://mh5_description/meshes/left_lower_arm.dae
- link left_upper_arm: geometry collision mesh filename=package://mh5_description/meshes/upper_arm.dae; visual mesh filename=package://mh5_description/meshes/upper_arm.dae
- link right_foot: geometry collision mesh filename=package://mh5_description/meshes/foot_revH.dae; visual mesh filename=package://mh5_description/meshes/foot_revH.dae
- link right_gripper: geometry collision mesh filename=package://mh5_description/meshes/gripper.dae; visual mesh filename=package://mh5_description/meshes/gripper.dae
- link right_lower_arm: geometry collision mesh filename=package://mh5_description/meshes/right_lower_arm.dae; visual mesh filename=package://mh5_description/meshes/right_lower_arm.dae
- link right_upper_arm: geometry collision mesh filename=package://mh5_description/meshes/upper_arm.dae; visual mesh filename=package://mh5_description/meshes/upper_arm.dae
